File: Group_07.brd (EAGLE design)
At the start: 62.2 x 74.9 mm, 29 parts, among them J1 POWER_JACKPTH_LOCK, U1 +12v, U3 TCA9546ASO16, U4 TMUX1208

Commit message: risoluzione conflitti drc MD S.R.L.
Routing:
- net GND: track 231.1 -> 267.1 mm, vias 4 -> 6
Changed lines of the file:
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@@
 <wire x1="52.324" y1="27.94" x2="46.609" y2="27.94" width="0.254" layer="1"/>
 <wire x1="46.609" y1="27.94" x2="45.5295" y2="26.8605" width="0.254" layer="1"/>
-<wire x1="45.5295" y1="26.8605" x2="45.466" y2="26.797" width="0.254" layer="1"/>
 <wire x1="45.5295" y1="26.8605" x2="44.196" y2="28.194" width="0.254" layer="1"/>
 <wire x1="44.196" y1="56.769" x2="44.3484" y2="56.9214" width="0.254" layer="1"/>
@@
 <wire x1="5.588" y1="8.763" x2="5.588" y2="8.1534" width="0.254" layer="1"/>
 <wire x1="5.588" y1="8.1534" x2="17.3133375" y2="8.1534" width="0.254" layer="1"/>
-<wire x1="19.431" y1="6.096" x2="19.3707375" y2="6.096" width="0.254" layer="1"/>
 <wire x1="17.3133375" y1="8.1534" x2="19.3707375" y2="6.096" width="0.254" layer="1"/>
 <wire x1="19.3707375" y1="6.096" x2="19.9313375" y2="5.5354" width="0.254" layer="1"/>
@@
 <wire x1="47.412" y1="13.4776" x2="47.412" y2="16.531" width="0.254" layer="1"/>
 <wire x1="44.323" y1="2.413" x2="44.577" y2="2.667" width="0.254" layer="1"/>
-<wire x1="47.412" y1="16.531" x2="50.662" y2="16.531" width="0" layer="19" extent="1-1"/>
+<wire x1="47.5576" y1="17.39673125" x2="47.72126875" y2="17.5604" width="0.254" layer="1"/>
+<wire x1="50.35273125" y1="17.5604" x2="50.5164" y2="17.39673125" width="0.254" layer="1"/>
+<wire x1="47.72126875" y1="17.5604" x2="50.35273125" y2="17.5604" width="0.254" layer="1"/>
+<wire x1="47.412" y1="16.531" x2="47.5576" y2="16.6766" width="0.254" layer="1"/>
+<wire x1="47.5576" y1="16.6766" x2="47.5576" y2="17.39673125" width="0.254" layer="1"/>
+<wire x1="50.5164" y1="17.39673125" x2="50.5164" y2="16.6766" width="0.254" layer="1"/>
+<wire x1="50.5164" y1="16.6766" x2="50.662" y2="16.531" width="0.254" layer="1"/>
+<wire x1="50.662" y1="16.531" x2="52.049" y2="16.531" width="0.254" layer="1"/>
+<wire x1="52.049" y1="16.531" x2="52.07" y2="16.51" width="0.254" layer="1"/>
+<via x="52.07" y="16.51" extent="1-16" drill="0.35"/>
+<wire x1="52.07" y1="16.51" x2="50.8" y2="17.78" width="0.254" layer="16"/>
+<wire x1="50.8" y1="17.78" x2="50.8" y2="29.21" width="0.254" layer="16"/>
+<via x="50.8" y="29.21" extent="1-16" drill="0.35"/>
+<wire x1="50.8" y1="29.21" x2="51.054" y2="29.464" width="0.254" layer="1"/>
+<wire x1="51.054" y1="29.464" x2="52.2572625" y2="29.464" width="0.254" layer="1"/>
+<wire x1="52.6796" y1="29.8863375" x2="52.6796" y2="32.9343375" width="0.254" layer="1"/>
+<wire x1="52.6796" y1="32.9343375" x2="53.1716625" y2="33.4264" width="0.254" layer="1"/>
+<wire x1="59.7662" y1="32.5090125" x2="59.7662" y2="31.4989875" width="0.254" layer="1"/>
+<wire x1="58.8488125" y1="33.4264" x2="59.7662" y2="32.5090125" width="0.254" layer="1"/>
+<wire x1="59.7662" y1="31.4989875" x2="58.547" y2="30.2797875" width="0.254" layer="1"/>
+<wire x1="58.547" y1="30.2797875" x2="58.547" y2="29.464" width="0.254" layer="1"/>
+<wire x1="52.2572625" y1="29.464" x2="52.6796" y2="29.8863375" width="0.254" layer="1"/>
+<wire x1="53.1716625" y1="33.4264" x2="58.8488125" y2="33.4264" width="0.254" layer="1"/>
 </signal>
 <signal name="12V">

Commit message: Modifiche traces GND
Routing:
- net GND: track 267.1 -> 90.7 mm, vias 6 -> 2
- net 5V: track 281.4 -> 255.3 mm, vias 15 -> 17
- net N$1: track 12.7 -> 14.4 mm
- net 12V: track 11.3 -> 12.6 mm
- net N$17: track 12.8 -> 14.0 mm
- net TEMP_OUT: track 15.7 -> 16.8 mm
- net N$15: track 17.8 -> 18.8 mm
